Commit message: Added materials to the ground. Finished messing with inertia matrices.

File: urdf/gogoro.urdf (robot description, URDF)
Before this commit: robot gogoro, 4 links, 3 joints
Links:
- link back: mass 2.753e+00 -> 0.1
- link body: mass 6.5007e+01 -> 79.2
- link head: mass 8.280e+00 -> 0.1
Joints:
- joint front_wheel_joint: limit effort=0 velocity=100000 -> effort=0 velocity=1000

Commit message: Added Thormang3 description files to remove its dependency. Removed collision from everything except wheels and handlebar.

File: urdf/gogoro.urdf (robot description, URDF)
Before this commit: robot gogoro, 4 links, 3 joints
Links:
- link body: geometry visual mesh filename=package://gogoro_description/meshes/body.stl scale=0.001 0.001 0.001

File: urdf/thormang3_gogoro.xacro (robot description, xacro)
@@ -5,11 +5,11 @@
   <xacro:property name="pi" value="3.141592654" />
   <!-- Import all Gazebo-customization elements, including Gazebo colors -->
-  <xacro:include filename="$(find thormang3_description)/urdf/thormang3.gazebo" />
+  <xacro:include filename="$(find gogoro_description)/urdf/thormang3/thormang3.gazebo" />
   <!-- Import Rviz colors -->
-  <xacro:include filename="$(find thormang3_description)/urdf/materials.xacro" />
-  <xacro:include filename="$(find thormang3_description)/urdf/thormang3.structure.arm.xacro" />
-  <xacro:include filename="$(find thormang3_description)/urdf/thormang3.structure.leg.xacro" />
-  <xacro:include filename="$(find thormang3_description)/urdf/thormang3.structure.head.xacro" />
-  <xacro:include filename="$(find thormang3_description)/urdf/thormang3.transmissions.xacro" />
+  <xacro:include filename="$(find gogoro_description)/urdf/thormang3/materials.xacro" />
+  <xacro:include filename="$(find gogoro_description)/urdf/thormang3/thormang3.structure.arm.xacro" />
+  <xacro:include filename="$(find gogoro_description)/urdf/thormang3/thormang3.structure.leg.xacro" />
+  <xacro:include filename="$(find gogoro_description)/urdf/thormang3/thormang3.structure.head.xacro" />
+  <xacro:include filename="$(find gogoro_description)/urdf/thormang3/thormang3.transmissions.xacro" />
   <!-- Used for fixing robot -->
 <!--
@@ -31,4 +31,5 @@
   <!-- pelvis_link -->
   <link name="pelvis_link">
+    <!--
     <collision>
       <origin xyz="-0.01 0 0.07" rpy="0 0 0"/>
@@ -37,8 +38,9 @@
       </geometry>
     </collision>
+    -->
     <visual>
       <origin xyz="0 0 0" rpy="0 0 0"/>
       <geometry>
-        <mesh filename="package://thormang3_description/meshes/robotis_pelvis_link.stl" scale="0.001 0.001 0.001"/>
+          <mesh filename="package://gogoro_description/meshes/thormang3/robotis_pelvis_link.stl" scale="0.001 0.001 0.001"/>
       </geometry>
       <material name="grey"/>
@@ -63,4 +65,5 @@
   <!-- chest_link -->
   <link name="chest_link">
+    <!--
     <collision>
       <origin xyz="-0.01 0 0.11" rpy="0 0 0"/>
@@ -69,8 +72,9 @@
       </geometry>
     </collision>
+    -->
     <visual>
       <origin xyz="0 0 0" rpy="0 0 0"/>
       <geometry>
-        <mesh filename="package://thormang3_description/meshes/robotis_chest_link.stl" scale="0.001 0.001 0.001"/>
+          <mesh filename="package://gogoro_description/meshes/thormang3/robotis_chest_link.stl" scale="0.001 0.001 0.001"/>
       </geometry>
       <material name="grey"/>

Commit message: Changed ground material and PID values.

File: urdf/gogoro.urdf (robot description, URDF)
Before this commit: robot gogoro, 4 links, 3 joints
Joints:
- joint front_wheel_joint: limit effort=0 velocity=1000 -> (none)
